Commit message: Move URDF changes

File: models/movo_description/movo.urdf (robot description, URDF)
Before this commit: robot movo, 50 links, 49 joints
Links:
- link base_chassis_link: geometry collision mesh filename=../movo_description/meshes/movo_components/collision/vector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; visual mesh filename=../movo_description/meshes/movo_components/visual/vector_ba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
- link front_laser_link: geometry collision box size=0.1 0.1 0.1; visual mesh filename=../movo_description/meshes/sensors/visual/sick_tim.dae
- link kinect2_link: geometry collision mesh filename=../movo_description/meshes/sensors/collision/kinect_one_col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; visual mesh filename=../movo_description/meshes/sensors/visual/kinect_one.dae
- link left_arm_half_1_link: geometry collision mesh filename=../movo_description/meshes/manipulation/jaco/collision/arm_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; visual mesh filename=../movo_description/meshes/manipulation/jaco/visual/arm_hal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
- link left_arm_half_2_link: geometry collision mesh filename=../movo_description/meshes/manipulation/jaco/collision/arm_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; visual mesh filename=../movo_description/meshes/manipulation/jaco/visual/arm_hal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
- link left_base_link: geometry collision mesh filename=../movo_description/meshes/manipulation/jaco/collision/base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; visual mesh filename=../movo_description/meshes/manipulation/jaco/visual/base.dae
- link left_forearm_link: geometry collision mesh filename=../movo_description/meshes/manipulation/jaco/collision/fore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; visual mesh filename=../movo_description/meshes/manipulation/jaco/visual/forearm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
- link left_gripper_base_link: geometry collision mesh filename=../movo_description/meshes/manipulation/kinova_grippers/col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; visual mesh filename=../movo_description/meshes/manipulation/kinova_grippers/vis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
- link left_gripper_finger1_finger_tip_link: geometry collision mesh filename=../movo_description/meshes/manipulation/kinova_grippers/col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; visual mesh filename=../movo_description/meshes/manipulation/kinova_grippers/vis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
- link left_gripper_finger1_knuckle_link: geometry collision mesh filename=../movo_description/meshes/manipulation/kinova_grippers/col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; visual mesh filename=../movo_description/meshes/manipulation/kinova_grippers/vis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
- link left_gripper_finger2_finger_tip_link: geometry collision mesh filename=../movo_description/meshes/manipulation/kinova_grippers/col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; visual mesh filename=../movo_description/meshes/manipulation/kinova_grippers/vis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
- link left_gripper_finger2_knuckle_link: geometry collision mesh filename=../movo_description/meshes/manipulation/kinova_grippers/col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; visual mesh filename=../movo_description/meshes/manipulation/kinova_grippers/vis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
- link left_gripper_finger3_finger_tip_link: geometry collision mesh filename=../movo_description/meshes/manipulation/kinova_grippers/col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; visual mesh filename=../movo_description/meshes/manipulation/kinova_grippers/vis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
- link left_gripper_finger3_knuckle_link: geometry collision mesh filename=../movo_description/meshes/manipulation/kinova_grippers/col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; visual mesh filename=../movo_description/meshes/manipulation/kinova_grippers/vis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
- link left_shoulder_link: geometry collision mesh filename=../movo_description/meshes/manipulation/jaco/collision/shou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; visual mesh filename=../movo_description/meshes/manipulation/jaco/visual/shoulde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
- link left_wrist_3_link: geometry collision mesh filename=../movo_description/meshes/manipulation/jaco/collision/kino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; visual mesh filename=../movo_description/meshes/manipulation/jaco/visual/kinova_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
- link left_wrist_spherical_1_link: geometry collision mesh filename=../movo_description/meshes/manipulation/jaco/collision/wris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; visual mesh filename=../movo_description/meshes/manipulation/jaco/visual/wrist_s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
- link left_wrist_spherical_2_link: geometry collision mesh filename=../movo_description/meshes/manipulation/jaco/collision/wris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; visual mesh filename=../movo_description/meshes/manipulation/jaco/visual/wrist_s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
- link linear_actuator_fixed_link: geometry collision mesh filename=../movo_description/meshes/movo_components/collision/movo_f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; visual mesh filename=../movo_description/meshes/movo_components/visual/movo_fixe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
- link linear_actuator_link: geometry collision mesh filename=../movo_description/meshes/movo_components/collision/movo_u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; visual mesh filename=../movo_description/meshes/movo_components/visual/movo_movi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
- link lower_body_link: geometry visual mesh filename=../movo_description/meshes/movo_body/movo_lower_body.dae
- link mid_body_link: geometry visual mesh filename=../movo_description/meshes/movo_body/movo_mid_body.dae
- link pan_base_link: geometry collision mesh filename=../movo_description/meshes/pan_tilt/collision/pan_tilt_base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; visual mesh filename=../movo_description/meshes/pan_tilt/visual/pan_tilt_base.dae
- link pan_link: geometry collision mesh filename=../movo_description/meshes/pan_tilt/collision/pan_link.stl; visual mesh filename=../movo_description/meshes/pan_tilt/visual/pan_link.dae
- link rear_laser_link: geometry collision box size=0.1 0.1 0.1; visual mesh filename=../movo_description/meshes/sensors/visual/sick_tim.dae
- link right_arm_half_1_link: geometry collision mesh filename=../movo_description/meshes/manipulation/jaco/collision/arm_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; visual mesh filename=../movo_description/meshes/manipulation/jaco/visual/arm_hal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
- link right_arm_half_2_link: geometry collision mesh filename=../movo_description/meshes/manipulation/jaco/collision/arm_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; visual mesh filename=../movo_description/meshes/manipulation/jaco/visual/arm_hal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
- link right_base_link: geometry collision mesh filename=../movo_description/meshes/manipulation/jaco/collision/base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; visual mesh filename=../movo_description/meshes/manipulation/jaco/visual/base.dae
- link right_forearm_link: geometry collision mesh filename=../movo_description/meshes/manipulation/jaco/collision/fore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; visual mesh filename=../movo_description/meshes/manipulation/jaco/visual/forearm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
- link right_gripper_base_link: geometry collision mesh filename=../movo_description/meshes/manipulation/kinova_grippers/col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; visual mesh filename=../movo_description/meshes/manipulation/kinova_grippers/vis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
- link right_gripper_finger1_finger_tip_link: geometry collision mesh filename=../movo_description/meshes/manipulation/kinova_grippers/col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; visual mesh filename=../movo_description/meshes/manipulation/kinova_grippers/vis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
- link right_gripper_finger1_knuckle_link: geometry collision mesh filename=../movo_description/meshes/manipulation/kinova_grippers/col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; visual mesh filename=../movo_description/meshes/manipulation/kinova_grippers/vis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
- link right_gripper_finger2_finger_tip_link: geometry collision mesh filename=../movo_description/meshes/manipulation/kinova_grippers/col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; visual mesh filename=../movo_description/meshes/manipulation/kinova_grippers/vis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
- link right_gripper_finger2_knuckle_link: geometry collision mesh filename=../movo_description/meshes/manipulation/kinova_grippers/col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; visual mesh filename=../movo_description/meshes/manipulation/kinova_grippers/vis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
- link right_gripper_finger3_finger_tip_link: geometry collision mesh filename=../movo_description/meshes/manipulation/kinova_grippers/col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; visual mesh filename=../movo_description/meshes/manipulation/kinova_grippers/vis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
- link right_gripper_finger3_knuckle_link: geometry collision mesh filename=../movo_description/meshes/manipulation/kinova_grippers/col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; visual mesh filename=../movo_description/meshes/manipulation/kinova_grippers/vis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
- link right_shoulder_link: geometry collision mesh filename=../movo_description/meshes/manipulation/jaco/collision/shou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; visual mesh filename=../movo_description/meshes/manipulation/jaco/visual/shoulde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
- link right_wrist_3_link: geometry collision mesh filename=../movo_description/meshes/manipulation/jaco/collision/kino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; visual mesh filename=../movo_description/meshes/manipulation/jaco/visual/kinova_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
- link right_wrist_spherical_1_link: geometry collision mesh filename=../movo_description/meshes/manipulation/jaco/collision/wris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; visual mesh filename=../movo_description/meshes/manipulation/jaco/visual/wrist_s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
- link right_wrist_spherical_2_link: geometry collision mesh filename=../movo_description/meshes/manipulation/jaco/collision/wris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; visual mesh filename=../movo_description/meshes/manipulation/jaco/visual/wrist_s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
- link tilt_link: geometry collision mesh filename=../movo_description/meshes/pan_tilt/collision/tilt_link.stl; visual mesh filename=../movo_description/meshes/pan_tilt/visual/tilt_link.dae
- link upper_body_link: geometry visual mesh filename=../movo_description/meshes/movo_body/movo_upper_body.dae

Commit message: Movo path

File: models/movo_description/movo.urdf (robot description, URDF)
Before this commit: robot movo, 50 links, 49 joints
Links:
- link base_chassis_link: geometry collision mesh filename=meshes/movo_components/collision/vector_base_collision.stl; visual mesh filename=meshes/movo_components/visual/vector_base.dae
- link front_laser_link: geometry collision box size=0.1 0.1 0.1; visual mesh filename=meshes/sensors/visual/sick_tim.dae
- link kinect2_link: geometry collision mesh filename=meshes/sensors/collision/kinect_one_collision.stl; visual mesh filename=meshes/sensors/visual/kinect_one.dae
- link left_arm_half_1_link: geometry collision mesh filename=meshes/manipulation/jaco/collision/arm_half_1.stl; visual mesh filename=meshes/manipulation/jaco/visual/arm_half_1.dae
- link left_arm_half_2_link: geometry collision mesh filename=meshes/manipulation/jaco/collision/arm_half_2.stl; visual mesh filename=meshes/manipulation/jaco/visual/arm_half_2.dae
- link left_base_link: geometry collision mesh filename=meshes/manipulation/jaco/collision/base.stl; visual mesh filename=meshes/manipulation/jaco/visual/base.dae
- link left_forearm_link: geometry collision mesh filename=meshes/manipulation/jaco/collision/forearm_7dof.stl; visual mesh filename=meshes/manipulation/jaco/visual/forearm_7dof.dae
- link left_gripper_base_link: geometry collision mesh filename=meshes/manipulation/kinova_grippers/collision/kg3_base_link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; visual mesh filename=meshes/manipulation/kinova_grippers/visual/kg3_base_link.dae
- link left_gripper_finger1_finger_tip_link: geometry collision mesh filename=meshes/manipulation/kinova_grippers/collision/finger_tip.stl; visual mesh filename=meshes/manipulation/kinova_grippers/visual/finger_tip.dae
- link left_gripper_finger1_knuckle_link: geometry collision mesh filename=meshes/manipulation/kinova_grippers/collision/finger_knuckl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; visual mesh filename=meshes/manipulation/kinova_grippers/visual/finger_knuckle.d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
- link left_gripper_finger2_finger_tip_link: geometry collision mesh filename=meshes/manipulation/kinova_grippers/collision/finger_tip.stl; visual mesh filename=meshes/manipulation/kinova_grippers/visual/finger_tip.dae
- link left_gripper_finger2_knuckle_link: geometry collision mesh filename=meshes/manipulation/kinova_grippers/collision/finger_knuckl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; visual mesh filename=meshes/manipulation/kinova_grippers/visual/finger_knuckle.d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
- link left_gripper_finger3_finger_tip_link: geometry collision mesh filename=meshes/manipulation/kinova_grippers/collision/finger_tip.stl; visual mesh filename=meshes/manipulation/kinova_grippers/visual/finger_tip.dae
- link left_gripper_finger3_knuckle_link: geometry collision mesh filename=meshes/manipulation/kinova_grippers/collision/finger_knuckl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; visual mesh filename=meshes/manipulation/kinova_grippers/visual/finger_knuckle.d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
- link left_shoulder_link: geometry collision mesh filename=meshes/manipulation/jaco/collision/shoulder_7dof.stl; visual mesh filename=meshes/manipulation/jaco/visual/shoulder_7dof.dae
- link left_wrist_3_link: geometry collision mesh filename=meshes/manipulation/jaco/collision/kinova_actuator_gearing.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; visual mesh filename=meshes/manipulation/jaco/visual/kinova_actuator_gearing.dae
- link left_wrist_spherical_1_link: geometry collision mesh filename=meshes/manipulation/jaco/collision/wrist_spherical_1.stl; visual mesh filename=meshes/manipulation/jaco/visual/wrist_spherical_1.dae
- link left_wrist_spherical_2_link: geometry collision mesh filename=meshes/manipulation/jaco/collision/wrist_spherical_2.stl; visual mesh filename=meshes/manipulation/jaco/visual/wrist_spherical_2.dae
- link linear_actuator_fixed_link: geometry collision mesh filename=meshes/movo_components/collision/movo_fixed_body_collision.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; visual mesh filename=meshes/movo_components/visual/movo_fixed_payload.dae
- link linear_actuator_link: geometry collision mesh filename=meshes/movo_components/collision/movo_upper_body_collision.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; visual mesh filename=meshes/movo_components/visual/movo_moving_payload.dae
- link lower_body_link: geometry visual mesh filename=meshes/movo_body/movo_lower_body.dae
- link mid_body_link: geometry visual mesh filename=meshes/movo_body/movo_mid_body.dae
- link pan_base_link: geometry collision mesh filename=meshes/pan_tilt/collision/pan_tilt_base.stl; visual mesh filename=meshes/pan_tilt/visual/pan_tilt_base.dae
- link pan_link: geometry collision mesh filename=meshes/pan_tilt/collision/pan_link.stl; visual mesh filename=meshes/pan_tilt/visual/pan_link.dae
- link rear_laser_link: geometry collision box size=0.1 0.1 0.1; visual mesh filename=meshes/sensors/visual/sick_tim.dae
- link right_arm_half_1_link: geometry collision mesh filename=meshes/manipulation/jaco/collision/arm_half_1.stl; visual mesh filename=meshes/manipulation/jaco/visual/arm_half_1.dae
- link right_arm_half_2_link: geometry collision mesh filename=meshes/manipulation/jaco/collision/arm_half_2.stl; visual mesh filename=meshes/manipulation/jaco/visual/arm_half_2.dae
- link right_base_link: geometry collision mesh filename=meshes/manipulation/jaco/collision/base.stl; visual mesh filename=meshes/manipulation/jaco/visual/base.dae
- link right_forearm_link: geometry collision mesh filename=meshes/manipulation/jaco/collision/forearm_7dof.stl; visual mesh filename=meshes/manipulation/jaco/visual/forearm_7dof.dae
- link right_gripper_base_link: geometry collision mesh filename=meshes/manipulation/kinova_grippers/collision/kg3_base_link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; visual mesh filename=meshes/manipulation/kinova_grippers/visual/kg3_base_link.dae
- link right_gripper_finger1_finger_tip_link: geometry collision mesh filename=meshes/manipulation/kinova_grippers/collision/finger_tip.stl; visual mesh filename=meshes/manipulation/kinova_grippers/visual/finger_tip.dae
- link right_gripper_finger1_knuckle_link: geometry collision mesh filename=meshes/manipulation/kinova_grippers/collision/finger_knuckl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; visual mesh filename=meshes/manipulation/kinova_grippers/visual/finger_knuckle.d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
- link right_gripper_finger2_finger_tip_link: geometry collision mesh filename=meshes/manipulation/kinova_grippers/collision/finger_tip.stl; visual mesh filename=meshes/manipulation/kinova_grippers/visual/finger_tip.dae
- link right_gripper_finger2_knuckle_link: geometry collision mesh filename=meshes/manipulation/kinova_grippers/collision/finger_knuckl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; visual mesh filename=meshes/manipulation/kinova_grippers/visual/finger_knuckle.d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
- link right_gripper_finger3_finger_tip_link: geometry collision mesh filename=meshes/manipulation/kinova_grippers/collision/finger_tip.stl; visual mesh filename=meshes/manipulation/kinova_grippers/visual/finger_tip.dae
- link right_gripper_finger3_knuckle_link: geometry collision mesh filename=meshes/manipulation/kinova_grippers/collision/finger_knuckl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; visual mesh filename=meshes/manipulation/kinova_grippers/visual/finger_knuckle.d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
- link right_shoulder_link: geometry collision mesh filename=meshes/manipulation/jaco/collision/shoulder_7dof.stl; visual mesh filename=meshes/manipulation/jaco/visual/shoulder_7dof.dae
- link right_wrist_3_link: geometry collision mesh filename=meshes/manipulation/jaco/collision/kinova_actuator_gearing.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; visual mesh filename=meshes/manipulation/jaco/visual/kinova_actuator_gearing.dae
- link right_wrist_spherical_1_link: geometry collision mesh filename=meshes/manipulation/jaco/collision/wrist_spherical_1.stl; visual mesh filename=meshes/manipulation/jaco/visual/wrist_spherical_1.dae
- link right_wrist_spherical_2_link: geometry collision mesh filename=meshes/manipulation/jaco/collision/wrist_spherical_2.stl; visual mesh filename=meshes/manipulation/jaco/visual/wrist_spherical_2.dae
- link tilt_link: geometry collision mesh filename=meshes/pan_tilt/collision/tilt_link.stl; visual mesh filename=meshes/pan_tilt/visual/tilt_link.dae
- link upper_body_link: geometry visual mesh filename=meshes/movo_body/movo_upper_body.dae
