Commit message: MOVO tool and base

File: models/movo_description/movo_robotiq.urdf (robot description, URDF)
Before this commit: robot movo, 53 links, 52 joints
Links:
- added link base_link_0
- added link base_link_1
- added link left_tool_link
- added link right_tool_link
- added link world_link
Joints:
- added joint left_tool_fixed_joint: type fixed, parent left_ee_link, child left_tool_link, origin xyz=0 0 0 rpy=1.570796325 0 1.570796325
- added joint right_tool_fixed_joint: type fixed, parent right_ee_link, child right_tool_link, origin xyz=0 0 0 rpy=1.570796325 0 1.570796325
- added joint theta: type continuous, parent base_link_1, child base_link, axis 0 0 1, limit effort=1000.0 velocity=1.5708
- added joint x: type prismatic, parent world_link, child base_link_0, axis 1 0 0, limit lower=-2.5 upper=2.5 effort=1000.0 velocity=1.0
- added joint y: type prismatic, parent base_link_0, child base_link_1, axis 0 1 0, limit lower=-2.5 upper=2.5 effort=1000.0 velocity=1.0
