Commit message: Collision MOVO

File: models/movo_description/movo_robotiq_collision.urdf (robot description, URDF)
Before this commit: robot movo, 58 links, 57 joints
Links:
- link base_chassis_link: geometry collision mesh filename=package://movo_description/meshes/movo_components/collision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; visual mesh filename=package://movo_description/meshes/movo_components/collision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
- link front_laser_link: geometry collision box size=0.1 0.1 0.1; visual box size=0.1 0.1 0.1
- link kinect2_link: geometry collision mesh filename=package://movo_description/meshes/sensors/collision/kinect_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; visual mesh filename=package://movo_description/meshes/sensors/collision/kinect_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
- link left_arm_half_1_link: geometry collision mesh filename=package://movo_description/meshes/manipulation/jaco/collisi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; visual mesh filename=package://movo_description/meshes/manipulation/jaco/collisi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
- link left_arm_half_2_link: geometry collision mesh filename=package://movo_description/meshes/manipulation/jaco/collisi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; visual mesh filename=package://movo_description/meshes/manipulation/jaco/collisi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
- link left_base_link: geometry collision mesh filename=package://movo_description/meshes/manipulation/jaco/collisi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; visual mesh filename=package://movo_description/meshes/manipulation/jaco/collisi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
- link left_forearm_link: geometry collision mesh filename=package://movo_description/meshes/manipulation/jaco/collisi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; visual mesh filename=package://movo_description/meshes/manipulation/jaco/collisi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
- link left_shoulder_link: geometry collision mesh filename=package://movo_description/meshes/manipulation/jaco/collisi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; visual mesh filename=package://movo_description/meshes/manipulation/jaco/collisi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
- link left_wrist_3_link: geometry collision mesh filename=package://movo_description/meshes/manipulation/jaco/collisi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; visual mesh filename=package://movo_description/meshes/manipulation/jaco/collisi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
- link left_wrist_spherical_1_link: geometry collision mesh filename=package://movo_description/meshes/manipulation/jaco/collisi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; visual mesh filename=package://movo_description/meshes/manipulation/jaco/collisi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
- link left_wrist_spherical_2_link: geometry collision mesh filename=package://movo_description/meshes/manipulation/jaco/collisi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; visual mesh filename=package://movo_description/meshes/manipulation/jaco/collisi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
- link linear_actuator_fixed_link: geometry collision mesh filename=package://movo_description/meshes/movo_components/collision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; visual mesh filename=package://movo_description/meshes/movo_components/collision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
- link linear_actuator_link: geometry collision mesh filename=package://movo_description/meshes/movo_components/collision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; visual mesh filename=package://movo_description/meshes/movo_components/collision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
- link pan_base_link: geometry collision mesh filename=package://movo_description/meshes/pan_tilt/collision/pan_ti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; visual mesh filename=package://movo_description/meshes/pan_tilt/collision/pan_ti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
- link pan_link: geometry collision mesh filename=package://movo_description/meshes/pan_tilt/collision/pan_li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; visual mesh filename=package://movo_description/meshes/pan_tilt/collision/pan_li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
- link rear_laser_link: geometry collision box size=0.1 0.1 0.1; visual box size=0.1 0.1 0.1
- link right_arm_half_1_link: geometry collision mesh filename=package://movo_description/meshes/manipulation/jaco/collisi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; visual mesh filename=package://movo_description/meshes/manipulation/jaco/collisi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
- link right_arm_half_2_link: geometry collision mesh filename=package://movo_description/meshes/manipulation/jaco/collisi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; visual mesh filename=package://movo_description/meshes/manipulation/jaco/collisi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
- link right_base_link: geometry collision mesh filename=package://movo_description/meshes/manipulation/jaco/collisi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; visual mesh filename=package://movo_description/meshes/manipulation/jaco/collisi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
- link right_forearm_link: geometry collision mesh filename=package://movo_description/meshes/manipulation/jaco/collisi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; visual mesh filename=package://movo_description/meshes/manipulation/jaco/collisi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
- link right_gripper_base_link: geometry collision mesh filename=package://movo_description/meshes/manipulation/robotiq/coll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; visual mesh filename=package://movo_description/meshes/manipulation/robotiq/coll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
- link right_gripper_finger1_finger_link: geometry collision mesh filename=package://movo_description/meshes/manipulation/robotiq/coll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; visual mesh filename=package://movo_description/meshes/manipulation/robotiq/coll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
- link right_gripper_finger1_finger_tip_link: geometry collision mesh filename=package://movo_description/meshes/manipulation/robotiq/coll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; visual mesh filename=package://movo_description/meshes/manipulation/robotiq/coll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
- link right_gripper_finger1_inner_knuckle_link: geometry collision mesh filename=package://movo_description/meshes/manipulation/robotiq/coll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; visual mesh filename=package://movo_description/meshes/manipulation/robotiq/coll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
- link right_gripper_finger1_knuckle_link: geometry collision mesh filename=package://movo_description/meshes/manipulation/robotiq/coll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; visual mesh filename=package://movo_description/meshes/manipulation/robotiq/coll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
- link right_gripper_finger2_finger_link: geometry collision mesh filename=package://movo_description/meshes/manipulation/robotiq/coll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; visual mesh filename=package://movo_description/meshes/manipulation/robotiq/coll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
- link right_gripper_finger2_finger_tip_link: geometry collision mesh filename=package://movo_description/meshes/manipulation/robotiq/coll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; visual mesh filename=package://movo_description/meshes/manipulation/robotiq/coll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
- link right_gripper_finger2_inner_knuckle_link: geometry collision mesh filename=package://movo_description/meshes/manipulation/robotiq/coll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; visual mesh filename=package://movo_description/meshes/manipulation/robotiq/coll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
- link right_gripper_finger2_knuckle_link: geometry collision mesh filename=package://movo_description/meshes/manipulation/robotiq/coll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; visual mesh filename=package://movo_description/meshes/manipulation/robotiq/coll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
- link right_robotiq_coupler_link: geometry collision mesh filename=package://movo_description/meshes/manipulation/robotiq/coll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; visual mesh filename=package://movo_description/meshes/manipulation/robotiq/coll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
- link right_shoulder_link: geometry collision mesh filename=package://movo_description/meshes/manipulation/jaco/collisi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; visual mesh filename=package://movo_description/meshes/manipulation/jaco/collisi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
- link right_wrist_3_link: geometry collision mesh filename=package://movo_description/meshes/manipulation/jaco/collisi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; visual mesh filename=package://movo_description/meshes/manipulation/jaco/collisi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
- link right_wrist_spherical_1_link: geometry collision mesh filename=package://movo_description/meshes/manipulation/jaco/collisi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; visual mesh filename=package://movo_description/meshes/manipulation/jaco/collisi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
- link right_wrist_spherical_2_link: geometry collision mesh filename=package://movo_description/meshes/manipulation/jaco/collisi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; visual mesh filename=package://movo_description/meshes/manipulation/jaco/collisi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
- link tilt_link: geometry collision mesh filename=package://movo_description/meshes/pan_tilt/collision/tilt_l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; visual mesh filename=package://movo_description/meshes/pan_tilt/collision/tilt_l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
