Commit message: abb_irb_track double tool-ik transf corrected. Add agripper to irb_track test. Single-arm test added to eth_rfl.

File: models/abb_irb6600_track/urdf/irb6600_track.urdf (robot description, URDF)
Before this commit: robot abb_irb6600_track, 16 links, 15 joints
Links:
- added link eef_base_link; collision mesh filename=../meshes/eth_rfl_gripper/collision/eth_rfl_gripper_collisi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 scale=.001 .001 .001; visual mesh filename=../meshes/eth_rfl_gripper/visual/eth_rfl_gripper_visual.stl scale=.001 .001 .001
- added link eef_tcp_frame
Joints:
- added joint ee_to_robot: type fixed, parent robot_tool0, child eef_base_link, origin xyz=0 0 0 rpy=0 0 0
- added joint eef_base_to_tcp: type fixed, parent eef_base_link, child eef_tcp_frame, origin xyz=0.0 0.0 0.475 rpy=0 0 0

File: models/eth_rfl/urdf/eth_rfl.urdf (robot description, URDF)
Before this commit: robot eth_rfl, 19 links, 18 joints
Links:
- link eef_base_link: geometry collision mesh filename=../meshes/eth_rfl_gripper/collision/eth_rfl_gripper_collisi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 scale=.001 .001 .001; visual mesh filename=../meshes/eth_rfl_gripper/visual/eth_rfl_gripper_visual.stl scale=.001 .001 .001
Joints:
- joint eef_base_to_tcp: origin xyz=0.0 0.0 0 rpy=0 0 0 -> xyz=0.0 0.0 0.475 rpy=0 0 0
