Commit message: in the middle of getting eth_rfl_pick demo work. The tcp frame is not right.

File: models/eth_rfl/urdf/eth_rfl.urdf (robot description, URDF)
Before this commit: robot eth_rfl, 19 links, 18 joints
Links:
- link eef_base_link: geometry 
Joints:
- joint eef_base_to_tcp: origin xyz=0.0 0.0 0.475 rpy=1.57079632679 0.0 0 -> xyz=0.0 0.0 0 rpy=0 0 0
- joint gantry_x_joint: axis 1 0 0 -> (none); limit lower=0 upper=20 effort=1 velocity=1.5 -> (none); type prismatic -> fixed
- joint gantry_y_joint: axis 0 1 0 -> (none); limit lower=0 upper=12.673 effort=1 velocity=1.5 -> (none); type prismatic -> fixed

Commit message: change nameing of the right arm in the eth_rfl urdf. Fixed some joints var in the BodyPaths generating fns in kuka_primitives.

File: models/eth_rfl/urdf/eth_rfl.urdf (robot description, URDF)
Before this commit: robot eth_rfl, 19 links, 18 joints
Links:
- removed link eef_base_link
- removed link eef_tcp_frame
- removed link gantry_robot_mount
- removed link gantry_xy_carriage
- removed link robot_base
- removed link robot_base_link
- removed link robot_link_1
- removed link robot_link_2
- removed link robot_link_3
- removed link robot_link_4
- removed link robot_link_5
- removed link robot_link_6
- removed link robot_tool0
- added link gantry_r_robot_mount
- added link r_eef_base_link; collision mesh filename=../meshes/eth_rfl_gripper/collision/eth_rfl_gripper_collisi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 scale=.001 .001 .001; visual mesh filename=../meshes/eth_rfl_gripper/visual/eth_rfl_gripper_visual.stl scale=.001 .001 .001
- added link r_eef_tcp_frame
- added link r_gantry_xy_carriage; collision mesh filename=../meshes/eth_rfl_track/collision/eth_gudel_track_xy_carria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 scale=.001 .001 .001; visual mesh filename=../meshes/eth_rfl_track/visual/eth_gudel_track_xy_carriage_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 scale=.001 .001 .001
- added link r_robot_base
- added link r_robot_base_link; collision mesh filename=../meshes/irb4400l_30_243/collision/base_link.stl; visual mesh filename=../meshes/irb4400l_30_243/visual/base_link.stl
- added link r_robot_link_1; collision mesh filename=../meshes/irb4400l_30_243/collision/link_1.stl; visual mesh filename=../meshes/irb4400l_30_243/visual/link_1.stl
- added link r_robot_link_2; collision mesh filename=../meshes/irb4400l_30_243/collision/link_2.stl; visual mesh filename=../meshes/irb4400l_30_243/visual/link_2.stl
- added link r_robot_link_3; collision mesh filename=../meshes/irb4400l_30_243/collision/link_3.stl; visual mesh filename=../meshes/irb4400l_30_243/visual/link_3.stl
- added link r_robot_link_4; collision mesh filename=../meshes/irb4400l_30_243/collision/link_4.stl; visual mesh filename=../meshes/irb4400l_30_243/visual/link_4.stl
- added link r_robot_link_5; collision mesh filename=../meshes/irb4400l_30_243/collision/link_5.stl; visual mesh filename=../meshes/irb4400l_30_243/visual/link_5.stl
- added link r_robot_link_6; collision mesh filename=../meshes/irb4400l_30_243/collision/link_6.stl; visual mesh filename=../meshes/irb4400l_30_243/visual/link_6.stl
- added link r_robot_tool0
Joints:
- removed joint ee_to_robot
- removed joint eef_base_to_tcp
- removed joint robot_base_link-base
- removed joint robot_joint_1
- removed joint robot_joint_2
- removed joint robot_joint_3
- removed joint robot_joint_4
- removed joint robot_joint_5
- removed joint robot_joint_6
- removed joint robot_joint_6-tool0
- removed joint robot_to_gantry
- added joint r_ee_to_r_robot: type fixed, parent r_robot_tool0, child r_eef_base_link, origin xyz=0 0 0 rpy=0 1.57079632679 0
- added joint r_eef_base_to_tcp: type fixed, parent r_eef_base_link, child r_eef_tcp_frame, origin xyz=0.0 0.0 0.475 rpy=0 0 0
- added joint r_robot_base_link-base: type fixed, parent r_robot_base_link, child r_robot_base, origin xyz=0 0 0 rpy=0 0 0
- added joint r_robot_joint_1: type revolute, parent r_robot_base_link, child r_robot_link_1, origin xyz=0 0 0 rpy=0 0 0, axis 0 0 1, limit lower=-2.87979 upper=2.87979 effort=0 velocity=2.618
- added joint r_robot_joint_2: type revolute, parent r_robot_link_1, child r_robot_link_2, origin xyz=0.2 0 0.68 rpy=0 0 0, axis 0 1 0, limit lower=-1.2217 upper=1.658 effort=0 velocity=2.0944
- added joint r_robot_joint_3: type revolute, parent r_robot_link_2, child r_robot_link_3, origin xyz=0 0 0.89 rpy=0 0 0, axis 0 1 0, limit lower=-1.0472 upper=1.1345 effort=0 velocity=2.0944
- added joint r_robot_joint_4: type revolute, parent r_robot_link_3, child r_robot_link_4, origin xyz=1.38 0 0.15 rpy=0 0 0, axis 1 0 0, limit lower=-3.49 upper=3.49 effort=0 velocity=3.927
- added joint r_robot_joint_5: type revolute, parent r_robot_link_4, child r_robot_link_5, origin xyz=0 0 0 rpy=0 0 0, axis 0 1 0, limit lower=-2.0944 upper=2.0944 effort=0 velocity=4.3633
- added joint r_robot_joint_6: type revolute, parent r_robot_link_5, child r_robot_link_6, origin xyz=0 0 0 rpy=0 0 0, axis 1 0 0, limit lower=-6.9813 upper=6.9813 effort=0 velocity=5.7596
- added joint r_robot_joint_6-tool0: type fixed, parent r_robot_link_6, child r_robot_tool0, origin xyz=0.14 0 0 rpy=0 0 0
- added joint r_robot_to_gantry: type fixed, parent gantry_r_robot_mount, child r_robot_base_link, origin xyz=0 0 0 rpy=0 0 0
- joint gantry_x_joint: axis (none) -> 1 0 0; limit (none) -> lower=0 upper=20 effort=1 velocity=1.5; type fixed -> prismatic
- joint gantry_y_joint: axis (none) -> 0 1 0; child gantry_xy_carriage -> r_gantry_xy_carriage; limit (none) -> lower=0 upper=12.673 effort=1 velocity=1.5; type fixed -> prismatic
- joint gantry_z_carriage_mount: child gantry_robot_mount -> gantry_r_robot_mount
- joint gantry_z_joint: parent gantry_xy_carriage -> r_gantry_xy_carriage

Commit message: eth_rfl dual arms block pick test completed.

File: models/eth_rfl/urdf/eth_rfl.urdf (robot description, URDF)
Before this commit: robot eth_rfl, 19 links, 18 joints
Links:
- removed link gantry_r_robot_mount
- removed link gantry_z_carriage
- added link l_eef_base_link; collision mesh filename=../meshes/eth_rfl_gripper/collision/eth_rfl_gripper_collisi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 scale=.001 .001 .001; visual mesh filename=../meshes/eth_rfl_gripper/visual/eth_rfl_gripper_visual.stl scale=.001 .001 .001
- added link l_eef_tcp_frame
- added link l_gantry_robot_mount
- added link l_gantry_xy_carriage; collision mesh filename=../meshes/eth_rfl_track/collision/eth_gudel_track_xy_carria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 scale=.001 .001 .001; visual mesh filename=../meshes/eth_rfl_track/visual/eth_gudel_track_xy_carriage_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 scale=.001 .001 .001
- added link l_gantry_z_carriage; collision mesh filename=../meshes/eth_rfl_track/collision/eth_gudel_track_z_carriag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 scale=.001 .001 .001; visual mesh filename=../meshes/eth_rfl_track/visual/eth_gudel_track_z_carriage_v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 scale=.001 .001 .001
- added link l_robot_base
- added link l_robot_base_link; collision mesh filename=../meshes/irb4400l_30_243/collision/base_link.stl; visual mesh filename=../meshes/irb4400l_30_243/visual/base_link.stl
- added link l_robot_link_1; collision mesh filename=../meshes/irb4400l_30_243/collision/link_1.stl; visual mesh filename=../meshes/irb4400l_30_243/visual/link_1.stl
- added link l_robot_link_2; collision mesh filename=../meshes/irb4400l_30_243/collision/link_2.stl; visual mesh filename=../meshes/irb4400l_30_243/visual/link_2.stl
- added link l_robot_link_3; collision mesh filename=../meshes/irb4400l_30_243/collision/link_3.stl; visual mesh filename=../meshes/irb4400l_30_243/visual/link_3.stl
- added link l_robot_link_4; collision mesh filename=../meshes/irb4400l_30_243/collision/link_4.stl; visual mesh filename=../meshes/irb4400l_30_243/visual/link_4.stl
- added link l_robot_link_5; collision mesh filename=../meshes/irb4400l_30_243/collision/link_5.stl; visual mesh filename=../meshes/irb4400l_30_243/visual/link_5.stl
- added link l_robot_link_6; collision mesh filename=../meshes/irb4400l_30_243/collision/link_6.stl; visual mesh filename=../meshes/irb4400l_30_243/visual/link_6.stl
- added link l_robot_tool0
- added link r_gantry_robot_mount
- added link r_gantry_z_carriage; collision mesh filename=../meshes/eth_rfl_track/collision/eth_gudel_track_z_carriag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 scale=.001 .001 .001; visual mesh filename=../meshes/eth_rfl_track/visual/eth_gudel_track_z_carriage_v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 scale=.001 .001 .001
Joints:
- removed joint gantry_y_joint
- removed joint gantry_z_carriage_mount
- removed joint gantry_z_joint
- added joint l_ee_to_l_robot: type fixed, parent l_robot_tool0, child l_eef_base_link, origin xyz=0 0 0 rpy=0 1.57079632679 0
- added joint l_eef_base_to_tcp: type fixed, parent l_eef_base_link, child l_eef_tcp_frame, origin xyz=0.0 0.0 0.475 rpy=0 0 0
- added joint l_gantry_y_joint: type prismatic, parent gantry_y_bridge, child l_gantry_xy_carriage, origin xyz=0 12.673 0 rpy=0 0 0, axis 0 -1 0, limit lower=0 upper=12.673 effort=1 velocity=1.5
- added joint l_gantry_z_carriage_mount: type fixed, parent l_gantry_z_carriage, child l_gantry_robot_mount, origin xyz=0.545 -0.0075 -1.2 rpy=0 3.14159265359 0
- added joint l_gantry_z_joint: type prismatic, parent l_gantry_xy_carriage, child l_gantry_z_carriage, origin xyz=0 0 0 rpy=0 0 0, axis 0 0 -1, limit lower=0 upper=1.227 effort=1 velocity=1
- added joint l_robot_base_link-base: type fixed, parent l_robot_base_link, child l_robot_base, origin xyz=0 0 0 rpy=0 0 0
- added joint l_robot_joint_1: type revolute, parent l_robot_base_link, child l_robot_link_1, origin xyz=0 0 0 rpy=0 0 0, axis 0 0 1, limit lower=-2.87979 upper=2.87979 effort=0 velocity=2.618
- added joint l_robot_joint_2: type revolute, parent l_robot_link_1, child l_robot_link_2, origin xyz=0.2 0 0.68 rpy=0 0 0, axis 0 1 0, limit lower=-1.2217 upper=1.658 effort=0 velocity=2.0944
- added joint l_robot_joint_3: type revolute, parent l_robot_link_2, child l_robot_link_3, origin xyz=0 0 0.89 rpy=0 0 0, axis 0 1 0, limit lower=-1.0472 upper=1.1345 effort=0 velocity=2.0944
- added joint l_robot_joint_4: type revolute, parent l_robot_link_3, child l_robot_link_4, origin xyz=1.38 0 0.15 rpy=0 0 0, axis 1 0 0, limit lower=-3.49 upper=3.49 effort=0 velocity=3.927
- added joint l_robot_joint_5: type revolute, parent l_robot_link_4, child l_robot_link_5, origin xyz=0 0 0 rpy=0 0 0, axis 0 1 0, limit lower=-2.0944 upper=2.0944 effort=0 velocity=4.3633
- added joint l_robot_joint_6: type revolute, parent l_robot_link_5, child l_robot_link_6, origin xyz=0 0 0 rpy=0 0 0, axis 1 0 0, limit lower=-6.9813 upper=6.9813 effort=0 velocity=5.7596
- added joint l_robot_joint_6-tool0: type fixed, parent l_robot_link_6, child l_robot_tool0, origin xyz=0.14 0 0 rpy=0 0 0
- added joint l_robot_to_gantry: type fixed, parent l_gantry_robot_mount, child l_robot_base_link, origin xyz=0 0 0 rpy=0 0 0
- added joint r_gantry_y_joint: type prismatic, parent gantry_y_bridge, child r_gantry_xy_carriage, origin xyz=0 0 0 rpy=0 0 0, axis 0 1 0, limit lower=0 upper=12.673 effort=1 velocity=1.5
- added joint r_gantry_z_carriage_mount: type fixed, parent r_gantry_z_carriage, child r_gantry_robot_mount, origin xyz=0.545 -0.0075 -1.2 rpy=0 3.14159265359 0
- added joint r_gantry_z_joint: type prismatic, parent r_gantry_xy_carriage, child r_gantry_z_carriage, origin xyz=0 0 0 rpy=0 0 0, axis 0 0 -1, limit lower=0 upper=1.227 effort=1 velocity=1
- joint r_robot_to_gantry: parent gantry_r_robot_mount -> r_gantry_robot_mount
