Commit message: Removing sensors

File: models/irobot.urdf (robot description, URDF)
Before this commit: robot iRobot, 11 links, 10 joints
Links:
- removed link camera_link
- removed link hokuyo_laser_link
- removed link imu_sensor_link
Joints:
- removed joint camera_sensor_joint
- removed joint hokuyo_laser_joint
- removed joint imu_sensor_joint
