Commit message: Adding new models

File: models/franka_description/robots/panda_arm_hand.urdf (robot description, URDF)
Before this commit: robot panda, 12 links, 11 joints
Links:
- added link tool_link
Joints:
- added joint tool_joint: type fixed, parent panda_link8, child tool_link, origin xyz=0.0 0 0.1 rpy=0 0 2.35619449019, axis 0 0 1
