Commit message: added official meshes and panda urdf

File: models/franka_description/robots/panda.urdf (robot description, URDF)
Before this commit: robot panda, 12 links, 11 joints
Links:
- added link panda_grasptarget, mass 0.0
- link panda_hand: mass None -> .81; geometry collision mesh filename=meshes/collision/hand.obj; visual mesh filename=meshes/visual/hand.obj
- link panda_leftfinger: mass None -> 0.1; geometry collision mesh filename=meshes/collision/finger.obj; visual mesh filename=meshes/visual/finger.obj
- link panda_link0: mass None -> 2.9; geometry collision mesh filename=meshes/collision/link0.obj; visual mesh filename=meshes/collision/link0.obj
- link panda_link1: mass None -> 2.7; geometry collision mesh filename=meshes/collision/link1.obj; visual mesh filename=meshes/visual/link1.obj
- link panda_link2: mass None -> 2.73; geometry collision mesh filename=meshes/collision/link2.obj; visual mesh filename=meshes/visual/link2.obj
- link panda_link3: mass None -> 2.04; geometry collision mesh filename=meshes/collision/link3.obj; visual mesh filename=meshes/visual/link3.obj
- link panda_link4: mass None -> 2.08; geometry collision mesh filename=meshes/collision/link4.obj; visual mesh filename=meshes/visual/link4.obj
- link panda_link5: mass None -> 3; geometry collision mesh filename=meshes/collision/link5.obj; visual mesh filename=meshes/visual/link5.obj
- link panda_link6: mass None -> 1.3; geometry collision mesh filename=meshes/collision/link6.obj; visual mesh filename=meshes/visual/link6.obj
- link panda_link7: mass None -> .2; geometry collision mesh filename=meshes/collision/link7.obj; visual mesh filename=meshes/collision/link7.obj
- link panda_link8: mass None -> 0.0
- link panda_rightfinger: mass None -> 0.1; geometry collision mesh filename=meshes/collision/finger.obj; visual mesh filename=meshes/visual/finger.obj
Joints:
- added joint panda_grasptarget_hand: type fixed, parent panda_hand, child panda_grasptarget, origin xyz=0 0 0.105 rpy=0 0 0
- joint panda_joint6: origin xyz=0 0 0 rpy=1.57079632679 0 0 -> xyz=0 0 0 rpy=0 0 0
- joint panda_joint7: origin xyz=0.088 0 0 rpy=1.57079632679 0 0 -> xyz=0.088 0 0 rpy=0 0 0

Commit message: panda kinematics updates, urdf updates

File: models/franka_description/robots/panda.urdf (robot description, URDF)
Before this commit: robot panda, 13 links, 12 joints
Joints:
- joint panda_finger_joint1: type prismatic -> fixed
- joint panda_finger_joint2: type prismatic -> fixed
- joint panda_joint7: origin xyz=0.088 0 0 rpy=0 0 0 -> xyz=0.088 0 0 rpy=1.57079632679 0 0
