Commit message: good planning for convex objects

File: models/franka_description/robots/panda_arm_hand_cam.urdf (robot description, URDF)
Before this commit: robot panda, 14 links, 13 joints
Joints:
- joint joint_dummy1: origin xyz=0.00000 0.00000 0.09000 rpy=0.00000 0.00000 0.00000 -> xyz=0.00000 0.00000 0.05000 rpy=0.00000 0.00000 0.00000
