Commit message: New wsg urdf

File: models/drake/wsg_50_description/urdf/wsg_50.urdf (robot description, URDF)
Before this commit: robot wsg_50, 5 links, 4 joints
Links:
- link base_link: geometry collision mesh filename=package://wsg_50_description/meshes/WSG50_110.stl scale=1 1 1; visual mesh filename=package://wsg_50_description/meshes/WSG50_110.stl scale=1 1 1
- link finger_left: geometry collision mesh filename=package://wsg_50_description/meshes/WSG-FMF.stl scale=0.001 0.001 0.001; visual mesh filename=package://wsg_50_description/meshes/WSG-FMF.stl scale=0.001 0.001 0.001
- link finger_right: geometry collision mesh filename=package://wsg_50_description/meshes/WSG-FMF.stl scale=0.001 0.001 0.001; visual mesh filename=package://wsg_50_description/meshes/WSG-FMF.stl scale=0.001 0.001 0.001
- link gripper_left: geometry collision mesh filename=package://wsg_50_description/meshes/GUIDE_WSG50_110.stl scale=0.001 0.001 0.001; visual mesh filename=package://wsg_50_description/meshes/GUIDE_WSG50_110.stl scale=0.001 0.001 0.001
- link gripper_right: geometry collision mesh filename=package://wsg_50_description/meshes/GUIDE_WSG50_110.stl scale=0.001 0.001 0.001; visual mesh filename=package://wsg_50_description/meshes/GUIDE_WSG50_110.stl scale=0.001 0.001 0.001
