Commit message: Grippers

File: models/drake/wsg_50_description/urdf/wsg_50_mesh_visual.urdf (robot description, URDF)
Before this commit: robot wsg_50, 6 links, 5 joints
Links:
- added link tool_link
Joints:
- added joint tool_joint: type fixed, parent wsg_50_base_link, child tool_link, origin xyz=0.0 0 0.125 rpy=0 0 1.57079632679, axis 0 0 1
- joint wsg_50_base_joint_gripper_left: axis 1 0 0 -> -1 0 0; limit lower=-0.055 upper=-0.0027 effort=1.0 velocity=1.0 -> lower=0.0027 upper=0.055 effort=1.0 velocity=1.0

File: models/franka_description/robots/hand.urdf (robot description, URDF)
Before this commit: robot hand, 3 links, 2 joints
Links:
- added link tool_link
Joints:
- added joint tool_joint: type fixed, parent panda_hand, child tool_link, origin xyz=0.0 0 0.1 rpy=0 0 1.57079632679, axis 0 0 1

Commit message: Changing table creation

File: models/drake/wsg_50_description/urdf/wsg_50_mesh_visual.urdf (robot description, URDF)
Before this commit: robot wsg_50, 7 links, 6 joints
Joints:
- joint tool_joint: origin xyz=0.0 0 0.125 rpy=0 0 1.57079632679 -> xyz=0.0 0 0.125 rpy=0 0 0
