Commit message: runs poorly

File: models/bi_panda/bi_panda.urdf (robot description, URDF)
Before this commit: robot bi_panda, 28 links, 27 joints
Joints:
- joint l_panda_joint0: origin xyz=-.4 .3 .05 rpy=0 0 0 -> xyz=-.6 .0 .05 rpy=0 0 0
- joint l_panda_joint6: origin xyz=0 0 0 rpy=0 0 0 -> xyz=0 0 0 rpy=1.57079632679 0 0
- joint r_panda_joint0: origin xyz=-.4 -.3 .05 rpy=0 0 0 -> xyz=-.4 -.6 .05 rpy=0 0 0

Commit message: revert urdf, update primitives, running better, still ofset from pick

File: models/bi_panda/bi_panda.urdf (robot description, URDF)
Before this commit: robot bi_panda, 28 links, 27 joints
Joints:
- joint bi_panda_base_joint: origin xyz=-.4 0 .05 rpy=0 0 0 -> xyz=0 0 0.5 rpy=0 0 0
- joint l_panda_joint0: origin xyz=-.6 .0 .05 rpy=0 0 0 -> xyz=-.3 0 0.05 rpy=0 0 0

Commit message: got pddlstream working with bi-panda

File: models/bi_panda/bi_panda.urdf (robot description, URDF)
Before this commit: robot bi_panda, 28 links, 27 joints
Joints:
- joint l_panda_joint0: origin xyz=-.3 0 0.05 rpy=0 0 0 -> xyz=-.3 0.4 0.05 rpy=0 0 0
- joint r_panda_joint0: origin xyz=-.4 -.6 .05 rpy=0 0 0 -> xyz=-.4 -.4 .05 rpy=0 0 0

Commit message: urdf updates, set up place to tray task

File: models/bi_panda/bi_panda.urdf (robot description, URDF)
Before this commit: robot bi_panda, 28 links, 27 joints
Joints:
- joint l_panda_joint0: origin xyz=-.3 0.4 0.05 rpy=0 0 0 -> xyz=0 0.5 0.05 rpy=0 0 0
- joint r_panda_joint0: origin xyz=-.4 -.4 .05 rpy=0 0 0 -> xyz=0 -.5 .05 rpy=0 0 0
- joint r_panda_joint6: origin xyz=0 0 0 rpy=0 0 0 -> xyz=0 0 0 rpy=1.57079632679 0 0
