Commit message: working with collisions, ignoring collisions for blocks other than when in collision with other blocks

File: models/bi_panda/bi_panda_shifted.urdf (robot description, URDF)
Before this commit: robot bi_panda, 28 links, 27 joints
Joints:
- joint l_panda_joint0: origin xyz=0 0.5 0.05 rpy=0 0 0 -> xyz=0 1 0.05 rpy=0 0 0

File: models/bi_panda/tray.urdf (robot description, URDF)
Before this commit: robot tray.urdf, 1 links, 0 joints
Links:
- link base_link: geometry collision box size=0.2 0.3 0.01; visual box size=0.3 0.4 0.01

Commit message: naive intelligent place working ignoring collisions

File: models/bi_panda/bi_panda_shifted.urdf (robot description, URDF)
Before this commit: robot bi_panda, 28 links, 27 joints
Joints:
- joint l_panda_joint0: origin xyz=0 1 0.05 rpy=0 0 0 -> xyz=0 1.05 0.05 rpy=0 0 0

File: models/bi_panda/tray.urdf (robot description, URDF)
Before this commit: robot tray, 1 links, 0 joints
Links:
- link base_link: mass 0.01 -> 0.1; geometry collision box size=0.2063 0.3143 0.0178; visual box size=0.2063 0.3143 0.0178

Commit message: more robust, broken trying to make traj more smooth

File: models/bi_panda/bi_panda_shifted.urdf (robot description, URDF)
Before this commit: robot bi_panda, 28 links, 27 joints
Joints:
- joint l_panda_joint0: origin xyz=0 1.05 0.05 rpy=0 0 0 -> xyz=0 .8 0.05 rpy=0 0 0
- joint r_panda_joint0: origin xyz=0 -.5 .05 rpy=0 0 0 -> xyz=0 -.3 .05 rpy=0 0 0

File: models/bi_panda/bi_panda_shifted_plate.urdf (robot description, URDF)
Before this commit: robot bi_panda, 26 links, 25 joints
Joints:
- joint l_panda_grasptarget_hand: origin xyz=0 0 0.105 rpy=0 0 0 -> xyz=0 0 0.25 rpy=0 0 0
- joint l_panda_joint0: origin xyz=0 1.05 0.05 rpy=0 0 0 -> xyz=0 .8 0.05 rpy=0 0 0

File: models/bi_panda/bin.urdf (robot description, URDF)
Before this commit: robot bin, 1 links, 0 joints
Links:
- link bin_body: geometry collision box size=0.01 0.35 0.17; collision box size=0.01 0.35 0.17

File: models/bi_panda/coke.urdf (robot description, URDF)
Before this commit: robot cylinder, 1 links, 0 joints
Links:
- link cylinder: mass 5 -> 2.5; geometry collision cylinder length=0.08 radius=0.015; visual cylinder length=0.08 radius=0.015

Commit message: updating

File: models/bi_panda/bi_panda_shifted.urdf (robot description, URDF)
Before this commit: robot bi_panda, 28 links, 27 joints
Joints:
- joint l_panda_joint1: limit lower=-2.9671 upper=2.9671 effort=87 velocity=2.1750 -> effort=87 velocity=2.1750

File: models/bi_panda/bi_panda_shifted_plate.urdf (robot description, URDF)
Before this commit: robot bi_panda, 26 links, 25 joints
Joints:
- joint l_panda_grasptarget_hand: origin xyz=0 0 0.25 rpy=0 0 0 -> xyz=0 0 0.19 rpy=0 0 0
- joint l_panda_joint0: origin xyz=0 .8 0.05 rpy=0 0 0 -> xyz=0 1.0 0.05 rpy=0 0 0
- joint l_panda_joint1: limit lower=-2.9671 upper=2.9671 effort=87 velocity=2.1750 -> effort=87 velocity=2.1750

File: models/bi_panda/bin.urdf (robot description, URDF)
Before this commit: robot bin, 1 links, 0 joints
Links:
- removed link bin_body
- added link body, mass 0.1; collision box size=0.01 0.35 0.17; collision box size=0.01 0.35 0.17

File: models/bi_panda/coke.urdf (robot description, URDF)
Before this commit: robot cylinder, 1 links, 0 joints
Links:
- link cylinder: mass 2.5 -> 1

File: models/bi_panda/tray.urdf (robot description, URDF)
Before this commit: robot tray, 1 links, 0 joints
Links:
- removed link base_link
- added link body, mass 0.1; collision box size=0.01 0.35 0.02; collision box size=0.01 0.35 0.02
