Commit message: testing moving the closer with a closer starting config

File: models/bi_panda/bi_panda_shifted_plate.urdf (robot description, URDF)
Before this commit: robot bi_panda, 26 links, 25 joints
Joints:
- joint l_panda_joint0: origin xyz=0 1.0 0.05 rpy=0 0 0 -> xyz=0 .9 0.05 rpy=0 0 0

Commit message: refactored to sample random y_distance for pre-determined range

File: models/bi_panda/bi_panda_shifted_plate.urdf (robot description, URDF)
Before this commit: robot bi_panda, 26 links, 25 joints
Joints:
- joint l_panda_grasptarget_hand: origin xyz=0 0 0.19 rpy=0 0 0 -> xyz=0 0 0.335 rpy=0 0 0
- joint l_panda_joint0: origin xyz=0 .9 0.05 rpy=0 0 0 -> xyz=0 .8 0.05 rpy=0 0 0
- joint r_panda_joint1: limit lower=-2.9671 upper=2.9671 effort=87 velocity=2.1750 -> lower=-2.4671 upper=2.9671 effort=87 velocity=2.1750

File: models/bi_panda/bin.urdf (robot description, URDF)
Before this commit: robot tray, 1 links, 0 joints
Links:
- link body: geometry collision box size=0.01 0.35 0.085; collision box size=0.01 0.35 0.085

File: models/bi_panda/coke.urdf (robot description, URDF)
Before this commit: robot cylinder, 1 links, 0 joints
Links:
- link cylinder: mass 1 -> 2; geometry collision cylinder length=0.05 radius=0.015; visual cylinder length=0.05 radius=0.015

File: models/bi_panda/tray.urdf (robot description, URDF)
Before this commit: robot tray, 1 links, 0 joints
Links:
- link body: geometry collision box size=0.01 0.35 0.02; collision box size=0.01 0.35 0.02
