Commit message: reconfig controller working

File: models/bi_panda/coke.urdf (robot description, URDF)
Before this commit: robot cylinder, 1 links, 0 joints
Links:
- link cylinder: mass 0.1 -> 2

Commit message: set up bin problem, set up baseline, problems with end goal placement and reconfig

File: models/bi_panda/coke.urdf (robot description, URDF)
Before this commit: robot cylinder, 1 links, 0 joints
Links:
- link cylinder: mass 2 -> 5; geometry collision cylinder length=0.08 radius=0.03; visual cylinder length=0.08 radius=0.03

File: models/bi_panda/tray.urdf (robot description, URDF)
Before this commit: robot tray, 1 links, 0 joints
Links:
- link base_link: mass 0.1 -> 0.01; geometry collision box size=0.2363 0.3143 0.0178; visual box size=0.2363 0.3143 0.0178

Commit message: commiting 70 percent success moving on

File: models/bi_panda/coke.urdf (robot description, URDF)
Before this commit: robot cylinder, 1 links, 0 joints
Links:
- link cylinder: mass 2 -> 2.5
